Commit message: Added UR5 integration with Husky. UR5 and Manipulator-H both now visible in RViz

File: husky-kinetic-devel/husky_description/urdf/decorations.urdf.xacro (robot description, xacro)
@@ -79,33 +79,36 @@
       <child link="rear_bumper_link" />
     </joint>
-    <xacro:if value="$(optenv HUSKY_TOP_PLATE_ENABLED true)">
-      <!-- Spawn the top plate -->
-      <link name="top_plate_link">
-        <visual>
-          <origin xyz="0 0 0" rpy="0 0 0" />
-          <geometry>
-            <mesh filename="package://husky_description/meshes/top_plate.dae" />
-          </geometry>
-        </visual>
-        <collision>
-          <origin xyz="0 0 0" rpy="0 0 0"/>
-          <geometry>
-            <mesh filename="package://husky_description/meshes/top_plate.dae" />
-          </geometry>
-        </collision>
-        <collision>
-          <!-- Extra collision tag for widgets on top plate -->
-          <geometry>
-            <box size="0.32 0.41 0.09" rpy="0 0 0"/>
-          </geometry>
-        </collision>
-      </link>
-      <!-- Attach top plate -->
-      <joint name="top_plate_joint" type="fixed">
-        <parent link="base_link" />
-        <child link="top_plate_link"/>
-        <origin xyz="0.0812 0 0.245" rpy="0 0 0"/>
-      </joint>
-    </xacro:if>
+    <!-- When the Robotis Manipulator-H is enabled, there is no top plate -->
+    <xacro:unless value="$(arg manipulator_h_enabled)">
+      <xacro:if value="$(optenv HUSKY_TOP_PLATE_ENABLED true)">
+        <!-- Spawn the top plate -->
+        <link name="top_plate_link">
+          <visual>
+            <origin xyz="0 0 0" rpy="0 0 0" />
+            <geometry>
+              <mesh filename="package://husky_description/meshes/top_plate.dae" />
+            </geometry>
+          </visual>
+          <collision>
+            <origin xyz="0 0 0" rpy="0 0 0"/>
+            <geometry>
+              <mesh filename="package://husky_description/meshes/top_plate.dae" />
+            </geometry>
+          </collision>
+          <collision>
+            <!-- Extra collision tag for widgets on top plate -->
+            <geometry>
+              <box size="0.32 0.41 0.09" rpy="0 0 0"/>
+            </geometry>
+          </collision>
+        </link>
+        <!-- Attach top plate -->
+        <joint name="top_plate_joint" type="fixed">
+          <parent link="base_link" />
+          <child link="top_plate_link"/>
+          <origin xyz="0.0812 0 0.245" rpy="0 0 0"/>
+        </joint>
+      </xacro:if>
+    </xacro:unless>
   </xacro:macro>
 </robot>

File: husky-kinetic-devel/husky_description/urdf/husky.urdf.xacro (robot description, xacro)
@@ -35,4 +35,6 @@
     <xacro:include filename="$(find manipulator_h_description)/urdf/manipulator_h.xacro" />
   </xacro:if>
+  <xacro:arg name="ur5_enabled" default="false"/> <!-- Added the UR5 -->
+  <xacro:include filename="$(find ur_description)/urdf/ur5.urdf.xacro" />
   <!-- Included URDF/XACRO Files -->
   <xacro:include filename="$(find husky_description)/urdf/decorations.urdf.xacro" />
@@ -138,4 +140,16 @@
     <xacro:kinect_camera prefix="camera" robot_namespace="$(arg robot_namespace)"/>
   </xacro:if>
+  <!-- Enable UR5 -->
+  <xacro:if value="$(arg ur5_enabled)">
+    <xacro:property name="reflect" value="-1" />
+    <!-- Spawn arm -->
+    <xacro:ur5_robot prefix="ur5_arm_" joint_limited="true"/>
+    <!-- Join arm -->
+    <joint name="ur5_arm_base" type="fixed">
+      <parent link="top_plate_link" />
+      <child link="ur5_arm_base_link" />
+      <origin xyz="0.3058 0 0.0065" rpy="0.0 0.0 -1.57" />
+    </joint>
+  </xacro:if>
   <!-- Enable Robotis Manipulator-H -->
   <xacro:if value="$(arg manipulator_h_enabled)">
