Commit message: Added the Manipulator-H to the Husky Kinetic package

File: husky-kinetic-devel/husky_description/urdf/husky.urdf.xacro (robot description, xacro)
@@ -30,4 +30,9 @@
   <xacro:arg name="robot_namespace" default="/" />
   <xacro:arg name="urdf_extras" default="empty.urdf" />
+  <xacro:arg name="manipulator_h_enabled" default="false"/> <!-- Added the Robotis Manipulator-H -->
+  <!-- Added the Robotis Manipulator-H -->
+  <xacro:if value="$(arg manipulator_h_enabled)">
+    <xacro:include filename="$(find manipulator_h_description)/urdf/manipulator_h.xacro" />
+  </xacro:if>
   <!-- Included URDF/XACRO Files -->
   <xacro:include filename="$(find husky_description)/urdf/decorations.urdf.xacro" />
@@ -133,4 +138,68 @@
     <xacro:kinect_camera prefix="camera" robot_namespace="$(arg robot_namespace)"/>
   </xacro:if>
+  <!-- Enable Robotis Manipulator-H -->
+  <xacro:if value="$(arg manipulator_h_enabled)">
+    <!--<xacro:property name="reflect" value="-1" />--> <!-- WHAT IS THIS???? -->
+    <!-- Box to simulate the base support -->
+    <link name="box">
+      <visual>
+        <origin xyz="0 0 0" />
+        <geometry>
+          <box size="0.225 0.42 0.202" />
+        </geometry>
+      </visual>
+    </link>
+    <gazebo reference="box">
+      <material>Gazebo/Orange</material>
+    </gazebo>
+    <!-- ZZZZZZZZZ -->
+    <!-- Husky's main chassis's height = +-24,6cm -->
+    <!-- Husky's manipulator h's support height = +- 20,2cm -->
+    <!-- The box's height is the same as the Husky's manipulator h's support height, so also 20,2cm -->
+    <!-- The center of the box is 20,2cm/2=10,1cm , so origin of the box height is 24,6 + 10,1 = 34,7cm -->
+    <!-- XXXXXXXXX -->
+    <!-- Husky's main chassis's length = 54,5cm . Half of the Husky is on positive "x" and the other half is on negative "x" -->
+    <!-- Box width is 22,5cm, so 54,5/2 - 22,5/2 = 16cm = 0,16m and 0,16m to the left, so -0,16m -> -0.162m actually -->
+    <!-- YYYYYYYYY -->
+    <!-- Husky's main chassis's width = 22,5cm, which is the same width as the box -->
+    <!-- Joint that connects the Husky's plate to the box -->
+    <joint name="box_base" type="fixed">
+      <parent link="base_link" />
+      <child link="box" />
+      <origin xyz="-0.162 0 0.347" rpy="0 0 0" />
+    </joint>
+    <!-- Cylinder to simulate the base of the manipulator -->
+    <link name="cylinder">
+      <visual>
+        <origin xyz="0 0 0" />
+        <geometry>
+          <cylinder length="0.0075" radius="0.08"/> <!-- Measurements not 100% accurate -->
+        </geometry>
+      </visual>
+    </link>
+    <gazebo reference="cylinder">
+      <material>Gazebo/Blue</material>
+    </gazebo>
+    <!-- ZZZZZZZZZ -->
+    <!-- The cylinder is on top of the box, so half of the height os the box above its center, plus half of the height of the cylinder = 10,475cm -->
+    <!-- XXXXXXXXX -->
+    <!-- The base of the manipulator has a length of 6,6cm and it's 2cm away from the end of the chassis, so the center of the manipulator in "x" is: -->
+    <!-- 22,5/2 - 6,6/2 - 2 = 5,95cm = 0,0595m and 0,0595m to the left, so -0,0595m -->
+    <!-- YYYYYYYYYY -->
+    <!-- The base of the manipulator has a width of 5,5cm and its a 11 cm away from the center of the box, so the center base is at: -->
+    <!-- 11 - 5,5/2 = 8,25cm = 0,0825m-->
+    <!-- Joint that connects the Husky's plate to the box -->
+    <joint name="cylinder_base" type="fixed">
+      <parent link="box" />
+      <child link="cylinder" />
+      <origin xyz="-0.0595 0.0825 0.10475" rpy="0 0 0" />
+    </joint>
+    <!-- Joint that connects the box to the arm -->
+    <joint name="manipulator_h_arm_base" type="fixed">
+      <parent link="cylinder" />
+      <child link="link1" />
+      <origin xyz="0 0 0.00375" rpy="0.0 0.0 1.57" />
+    </joint>
+  </xacro:if>
   <gazebo>
     <plugin name="gazebo_ros_control" filename="libgazebo_ros_control.so">

Commit message: Added the laser Hokuyo UST-10LX to the simulation (the one on top of the AGROB tower)

File: husky-kinetic-devel/husky_description/urdf/husky.urdf.xacro (robot description, xacro)
@@ -37,4 +37,5 @@
   <xacro:arg name="ur5_enabled" default="false"/> <!-- Added the UR5 -->
   <xacro:include filename="$(find ur_description)/urdf/ur5.urdf.xacro" />
+  <xacro:arg name="vertical_laser_enabled" default="false"/> <!-- Added the vertical laser Hokuyo UST-10LX -->
   <!-- Included URDF/XACRO Files -->
   <xacro:include filename="$(find husky_description)/urdf/decorations.urdf.xacro" />
@@ -216,4 +217,65 @@
     </joint>
   </xacro:if>
+  <!-- Added the vertical laser Hokuyo UST-10LX -->
+  <xacro:if value="$(arg vertical_laser_enabled)">
+    <link name="hokuyo_link">
+      <collision>
+        <origin xyz="0 0 0" rpy="0 0 0"/>
+        <geometry>
+	  <box size="0.001 0.001 0.001"/> <!-- Originally "0 0 0" but it causes Gazebo to crash -->
+        </geometry>
+      </collision>
+      <visual>
+        <origin xyz="0 0 0" rpy="0 0 0"/>
+        <geometry>
+          <mesh filename="package://husky_gazebo/meshes/hokuyo.dae"/> <!-- Previously using the file "hokuyo.dae" from the "robot_description" package inside the "agrob_simulator-master" package-->
+        </geometry>
+      </visual>
+      <inertial>
+        <mass value="1e-5" />
+        <origin xyz="0 0 0" rpy="0 0 0"/>
+        <inertia ixx="1e-5" ixy="0" ixz="0" iyy="1e-5" iyz="0" izz="1e-5" />
+      </inertial>
+    </link>
+    <gazebo reference="hokuyo_link">
+      <sensor name="laser" type="ray">
+        <pose>0.01 0 0.0175 0 0 0</pose>
+        <ray>
+          <scan>
+            <horizontal>
+              <samples>683</samples>
+              <resolution>1</resolution>
+              <min_angle>-2.09439510239</min_angle>
+              <max_angle>2.09439510239</max_angle>
+            </horizontal>
+          </scan>
+          <range>
+            <min>0.2</min>
+            <max>4</max>
+            <resolution>0.01</resolution>
+          </range>
+          <!--<noise>
+            <type>gaussian</type>
+            <mean>0.0</mean>
+            <stddev>0.01</stddev>
+          </noise>-->
+        </ray>
+        <plugin name="gazebo_ros_head_hokuyo_controller" filename="libgazebo_ros_laser.so">
+          <topicName>laser_vertical</topicName>
+          <frameName>hokuyo_link</frameName>
+        </plugin>
+        <always_on>1</always_on>
+        <update_rate>10</update_rate>
+        <visualize>true</visualize>
+      </sensor>
+    </gazebo>
+    <joint name="vertical_laser_base" type="fixed">
+      <origin
+        xyz="0.34 0.07 0.94"
+        rpy="0 1.33 0" /> <!-- Originally "0 1.33 -0.1" -->
+      <parent link="base_link" />
+      <child link="hokuyo_link" />
+    </joint>
+  </xacro:if>
   <gazebo>
     <plugin name="gazebo_ros_control" filename="libgazebo_ros_control.so">

Commit message: The colors of the cylinder and the box where the Manipulator-H is mounted are now visible in RViz. They used to be red

File: husky-kinetic-devel/husky_description/urdf/husky.urdf.xacro (robot description, xacro)
@@ -163,4 +163,7 @@
           <box size="0.225 0.42 0.202" />
         </geometry>
+        <material name="Gazebo/Orange_color">
+          <color rgba="1 0.5088 0.0468 1.0"/>
+        </material>
       </visual>
     </link>
@@ -191,4 +194,7 @@
           <cylinder length="0.0075" radius="0.08"/> <!-- Measurements not 100% accurate -->
         </geometry>
+        <material name="Gazebo/Blue_color">
+          <color rgba="0 0 1 1.0"/>
+        </material>
       </visual>
     </link>
