Commit message: Added "manipulator_h_gazebo" package and integrated it with MoveIt!. Simulated plans in RViz can now be executed and seen in Gazebo

File: manipulator_h_description/urdf/manipulator_h.xacro (robot description, xacro)
@@ -1,7 +1,6 @@
 <?xml version="1.0"?>
+<!-- NOTE: Changed "EffortJointInterface" to "PositionJointInterface" -->
 <!-- Revolute-Revolute Manipulator -->
 <robot name="robotis_manipulator_h" xmlns:xacro="http://www.ros.org/wiki/xacro">
-  <!-- some parameters -->
-  <xacro:property name="pi" value="3.141592654" />
   <!-- some parameters -->
   <xacro:property name="pi" value="3.141592654" />
@@ -53,8 +52,8 @@
     <type>transmission_interface/SimpleTransmission</type>
     <joint name="joint1">
-      <hardwareInterface>EffortJointInterface</hardwareInterface>
+      <hardwareInterface>hardware_interface/PositionJointInterface</hardwareInterface>
     </joint>
     <actuator name="motor1">
-      <hardwareInterface>EffortJointInterface</hardwareInterface>
+      <hardwareInterface>hardware_interface/PositionJointInterface</hardwareInterface>
       <mechanicalReduction>1</mechanicalReduction>
     </actuator>
@@ -95,8 +94,8 @@
     <type>transmission_interface/SimpleTransmission</type>
     <joint name="joint2">
-      <hardwareInterface>EffortJointInterface</hardwareInterface>
+      <hardwareInterface>hardware_interface/PositionJointInterface</hardwareInterface>
     </joint>
     <actuator name="motor2">
-      <hardwareInterface>EffortJointInterface</hardwareInterface>
+      <hardwareInterface>hardware_interface/PositionJointInterface</hardwareInterface>
       <mechanicalReduction>1</mechanicalReduction>
     </actuator>
@@ -137,8 +136,8 @@
     <type>transmission_interface/SimpleTransmission</type>
     <joint name="joint3">
-      <hardwareInterface>EffortJointInterface</hardwareInterface>
+      <hardwareInterface>hardware_interface/PositionJointInterface</hardwareInterface>
     </joint>
     <actuator name="motor3">
-      <hardwareInterface>EffortJointInterface</hardwareInterface>
+      <hardwareInterface>hardware_interface/PositionJointInterface</hardwareInterface>
       <mechanicalReduction>1</mechanicalReduction>
     </actuator>
@@ -179,8 +178,8 @@
     <type>transmission_interface/SimpleTransmission</type>
     <joint name="joint4">
-      <hardwareInterface>EffortJointInterface</hardwareInterface>
+      <hardwareInterface>hardware_interface/PositionJointInterface</hardwareInterface>
     </joint>
     <actuator name="motor4">
-      <hardwareInterface>EffortJointInterface</hardwareInterface>
+      <hardwareInterface>hardware_interface/PositionJointInterface</hardwareInterface>
       <mechanicalReduction>1</mechanicalReduction>
     </actuator>
@@ -221,8 +220,8 @@
     <type>transmission_interface/SimpleTransmission</type>
     <joint name="joint5">
-      <hardwareInterface>EffortJointInterface</hardwareInterface>
+      <hardwareInterface>hardware_interface/PositionJointInterface</hardwareInterface>
     </joint>
     <actuator name="motor5">
-      <hardwareInterface>EffortJointInterface</hardwareInterface>
+      <hardwareInterface>hardware_interface/PositionJointInterface</hardwareInterface>
       <mechanicalReduction>1</mechanicalReduction>
     </actuator>
@@ -263,8 +262,8 @@
     <type>transmission_interface/SimpleTransmission</type>
     <joint name="joint6">
-      <hardwareInterface>EffortJointInterface</hardwareInterface>
+      <hardwareInterface>hardware_interface/PositionJointInterface</hardwareInterface>
     </joint>
     <actuator name="motor6">
-      <hardwareInterface>EffortJointInterface</hardwareInterface>
+      <hardwareInterface>hardware_interface/PositionJointInterface</hardwareInterface>
       <mechanicalReduction>1</mechanicalReduction>
     </actuator>

Commit message: Added Husky packages to integrate the Manipulator-H with Husky in Gazebo

File: manipulator_h_description/urdf/manipulator_h.xacro (robot description, xacro)
@@ -2,19 +2,24 @@
 <!-- NOTE: Changed "EffortJointInterface" to "PositionJointInterface" -->
 <!-- Revolute-Revolute Manipulator -->
-<robot name="robotis_manipulator_h" xmlns:xacro="http://www.ros.org/wiki/xacro">
+<robot name="robotis_manipulator_h" xmlns:xacro="http://ros.org/wiki/xacro">
   <!-- some parameters -->
   <xacro:property name="pi" value="3.141592654" />
+  <!-- By default, do not enable Manipulator-H on top of the Husky -->
+  <xacro:arg name="manipulator_h_enabled" default="false" />
   <!-- Import all Gazebo-customization elements, including Gazebo colors -->
   <xacro:include filename="$(find manipulator_h_description)/urdf/manipulator_h.gazebo" />
   <!-- Import Rviz colors -->
   <xacro:include filename="$(find manipulator_h_description)/urdf/materials.xacro" />
+<!-- ///////////////////// IF HUSKY IS NOT CALLED, CREATE A LINK "world" TO CONNECT THE MANIPULATOR TO THE WORLD /////////////////// -->
   <!-- Used for fixing robot to Gazebo 'link 1' -->
-  <link name="world">
-  </link>
-  <joint name="world_fixed" type="fixed">
-    <origin xyz="0 0 0" rpy="0 0 0"/>
-    <parent link="world"/>
-    <child link="link1"/>
-  </joint>
+  <xacro:unless value="$(arg manipulator_h_enabled)">
+    <link name="world"/>
+    <joint name="world_fixed" type="fixed">
+      <origin xyz="0 0 0" rpy="0 0 0"/>
+      <parent link="world"/>
+      <child link="link1"/>
+    </joint>
+  </xacro:unless>
+<!-- /////////////////////////////////////////////////////////////////////////////////////////////////////////////////////////////// -->
   <!-- link 1 -->
   <link name="link1">

Commit message: MoveIt! now works with the real Robotis Manipulator-H (with some errors in the 5th joint). In simulation, started to implement the cutting tool but also with errors.

File: manipulator_h_description/urdf/manipulator_h.xacro (robot description, xacro)
@@ -255,44 +255,69 @@
     </inertial>
   </link>
-  <!-- Joint 6 -->
-  <joint name="joint6" type="revolute">
-    <parent link="link6"/>
-    <child link="end_link"/>
-    <origin xyz="0.12300 -0.04500 0.00000" rpy="0 0 0"/>
-    <axis xyz="1 0 0"/>
-    <limit velocity="6.5" effort="1000" lower="${-pi*0.5}" upper="${pi*0.5}" />
-    <dynamics damping="0.7"/>
-  </joint>
-  <transmission name="tran6">
-    <type>transmission_interface/SimpleTransmission</type>
-    <joint name="joint6">
-      <hardwareInterface>hardware_interface/EffortJointInterface</hardwareInterface>
-    </joint>
-    <actuator name="motor6">
-      <hardwareInterface>hardware_interface/EffortJointInterface</hardwareInterface>
-      <mechanicalReduction>1</mechanicalReduction>
-    </actuator>
-  </transmission>
-  <!-- end link -->
-  <link name="end_link">
-    <collision>
-      <origin xyz="0 0 0" rpy="0 0 0"/>
-      <geometry>
-        <mesh filename="package://manipulator_h_description/meshes/end_link.stl" scale="0.001 0.001 0.001"/>
-      </geometry>
-    </collision>
-    <visual>
-      <origin xyz="0 0 0" rpy="0 0 0"/>
-      <geometry>
-        <mesh filename="package://manipulator_h_description/meshes/end_link.stl" scale="0.001 0.001 0.001"/>
-      </geometry>
-      <material name="grey"/>
-    </visual>
-    <inertial>
-      <origin xyz="0.00337 0.00000 0.00000" rpy="0 0 0"/>
-      <mass value="0.01919"/>
-      <inertia ixx="1.0" ixy="0.0" ixz="0.0" iyy="1.0" iyz="0.0" izz="1.0" />
-      <!--<inertia ixx="0.00000938" ixy="0.0" ixz="0.0" iyy="0.00000338" iyz="0.0" izz="0.00000635" />-->
-    </inertial>
-  </link>
+  <!-- Default parts of the manipulator -->
+  <xacro:unless value="$(arg manipulator_h_enabled)">
+    <!-- Joint 6 -->
+    <joint name="joint6" type="revolute">
+      <parent link="link6"/>
+      <child link="end_link"/>
+      <origin xyz="0.12300 -0.04500 0.00000" rpy="0 0 0"/>
+      <axis xyz="1 0 0"/>
+      <limit velocity="6.5" effort="1000" lower="${-pi*0.5}" upper="${pi*0.5}" />
+      <dynamics damping="0.7"/>
+    </joint>
+    <transmission name="tran6">
+      <type>transmission_interface/SimpleTransmission</type>
+      <joint name="joint6">
+        <hardwareInterface>hardware_interface/EffortJointInterface</hardwareInterface>
+      </joint>
+      <actuator name="motor6">
+        <hardwareInterface>hardware_interface/EffortJointInterface</hardwareInterface>
+        <mechanicalReduction>1</mechanicalReduction>
+      </actuator>
+    </transmission>
+    <!-- end link -->
+    <link name="end_link">
+      <collision>
+        <origin xyz="0 0 0" rpy="0 0 0"/>
+        <geometry>
+          <mesh filename="package://manipulator_h_description/meshes/end_link.stl" scale="0.001 0.001 0.001"/>
+        </geometry>
+      </collision>
+      <visual>
+        <origin xyz="0 0 0" rpy="0 0 0"/>
+        <geometry>
+          <mesh filename="package://manipulator_h_description/meshes/end_link.stl" scale="0.001 0.001 0.001"/>
+        </geometry>
+        <material name="grey"/>
+      </visual>
+      <inertial>
+        <origin xyz="0.00337 0.00000 0.00000" rpy="0 0 0"/>
+        <mass value="0.01919"/>
+        <inertia ixx="1.0" ixy="0.0" ixz="0.0" iyy="1.0" iyz="0.0" izz="1.0" />
+        <!--<inertia ixx="0.00000938" ixy="0.0" ixz="0.0" iyy="0.00000338" iyz="0.0" izz="0.00000635" />-->
+      </inertial>
+    </link>
+  </xacro:unless>
+  <!-- Cutting tool loaded when Manipulator-H is on top of the Husky robot -->
+  <xacro:if value="$(arg manipulator_h_enabled)">
+    <joint name="joint6" type="revolute">
+      <origin xyz="0.32 -0.014 -0.021" rpy="0 0 0"/>
+      <axis xyz="1 0 0"/>
+      <parent link="link6"/>
+      <child link="cutting_tool"/>
+      <limit velocity="6.5" effort="1000" lower="${-pi*0.5}" upper="${pi*0.5}" />
+      <dynamics damping="0.7"/>
+    </joint>
+    <transmission name="tran6">
+      <type>transmission_interface/SimpleTransmission</type>
+      <joint name="joint6">
+        <hardwareInterface>hardware_interface/EffortJointInterface</hardwareInterface>
+      </joint>
+      <actuator name="motor6">
+        <hardwareInterface>hardware_interface/EffortJointInterface</hardwareInterface>
+        <mechanicalReduction>1</mechanicalReduction>
+      </actuator>
+    </transmission>
+    <xacro:include filename="$(find cutting_tool)/urdf/cutting_tool.urdf" />
+  </xacro:if>
 </robot>

Commit message: Added the cutting tool to the end as an and effector an now plans can be done with MoveIt!. Manipulator-H can now be planned with MoveIt! with no joint error. Coded plans still don't work.

File: manipulator_h_description/urdf/manipulator_h.xacro (robot description, xacro)
@@ -301,9 +301,10 @@
   <!-- Cutting tool loaded when Manipulator-H is on top of the Husky robot -->
   <xacro:if value="$(arg manipulator_h_enabled)">
+    <!-- Joint 6 -->
     <joint name="joint6" type="revolute">
-      <origin xyz="0.32 -0.014 -0.021" rpy="0 0 0"/>
+      <parent link="link6"/>
+      <child link="end_link"/>
+      <origin xyz="0.12300 -0.04500 0.00000" rpy="0 0 0"/>
       <axis xyz="1 0 0"/>
-      <parent link="link6"/>
-      <child link="cutting_tool"/>
       <limit velocity="6.5" effort="1000" lower="${-pi*0.5}" upper="${pi*0.5}" />
       <dynamics damping="0.7"/>
@@ -319,4 +320,42 @@
       </actuator>
     </transmission>
+    <!-- end link -->
+    <link name="end_link">
+      <collision>
+        <origin xyz="0 0 0" rpy="0 0 0"/>
+        <geometry>
+          <mesh filename="package://manipulator_h_description/meshes/end_link.stl" scale="0.001 0.001 0.001"/>
+        </geometry>
+      </collision>
+      <visual>
+        <origin xyz="0 0 0" rpy="0 0 0"/>
+        <geometry>
+          <mesh filename="package://manipulator_h_description/meshes/end_link.stl" scale="0.001 0.001 0.001"/>
+        </geometry>
+        <material name="grey"/>
+      </visual>
+      <inertial>
+        <origin xyz="0.00337 0.00000 0.00000" rpy="0 0 0"/>
+        <mass value="0.01919"/>
+        <inertia ixx="1.0" ixy="0.0" ixz="0.0" iyy="1.0" iyz="0.0" izz="1.0" />
+        <!--<inertia ixx="0.00000938" ixy="0.0" ixz="0.0" iyy="0.00000338" iyz="0.0" izz="0.00000635" />-->
+      </inertial>
+    </link>
+    <transmission name="tran6">
+      <type>transmission_interface/SimpleTransmission</type>
+      <joint name="joint6">
+        <hardwareInterface>hardware_interface/EffortJointInterface</hardwareInterface>
+      </joint>
+      <actuator name="motor6">
+        <hardwareInterface>hardware_interface/EffortJointInterface</hardwareInterface>
+        <mechanicalReduction>1</mechanicalReduction>
+      </actuator>
+    </transmission>
+    <joint name="joint7" type="fixed">
+      <origin xyz="0.2085 0.031 -0.018" rpy="0 0 0"/>
+      <axis xyz="1 0 0"/>
+      <parent link="end_link"/>
+      <child link="cutting_tool"/>
+    </joint>
     <xacro:include filename="$(find cutting_tool)/urdf/cutting_tool.urdf" />
   </xacro:if>
